Commit message: created a modular include for all sensors

File: model/robot.xacro (robot description, xacro)
@@ -74,4 +74,14 @@
         <color rgba="0.7 0.7 0.7 1"/>
     </material>
+<!-- Include the modular LIDAR sensor file -->
+<xacro:include filename="$(find mobile_dd_robot)/model/sensors/lidar.xacro" />
+<!-- Include the modular camera sensor file -->
+<xacro:include filename="$(find mobile_dd_robot)/model/sensors/camera.xacro" />
+<!-- Include the modular depth camera sensor file -->
+<xacro:include filename="$(find mobile_dd_robot)/model/sensors/depth_camera.xacro" />
+<!-- Include the modular IMU sensor file -->
+<xacro:include filename="$(find mobile_dd_robot)/model/sensors/imu.xacro" />
+<!-- Include the modular GPS sensor file -->
+<xacro:include filename="$(find mobile_dd_robot)/model/sensors/gps.xacro" />
 <!-- Over here we include the file that defines extra Gazebo options and motion control driver -->
 <xacro:include filename="$(find mobile_dd_robot)/model/robot.gazebo" />
@@ -202,200 +212,12 @@
 <!-- ########################################################### -->
 <!-- ########################################################### -->
-<!-- START: LIDAR connector and sensor										 -->
-<!-- ########################################################### -->
-<!-- LIDAR connector link -->
-<joint name="lidar_connector_joint" type="fixed">
-    <parent link="body_link"/>
-    <child link="lidar_connector_link"/>
-    <origin xyz="0 0 ${body_link_z_dim/2}" rpy="0 0 0"/>
-</joint>
-<link name="lidar_connector_link">
-    <visual>
-        <origin xyz="0 0 0" rpy="0 0 0"/>
-        <geometry>
-            <cylinder radius="0.02" length="0.06"/>
-        </geometry>
-        <material name="black"/>
-    </visual>
-    <collision>
-        <origin xyz="0 0 0" rpy="0 0 0"/>
-        <geometry>
-            <cylinder radius="0.02" length="0.06"/>
-        </geometry>
-    </collision>
-    <inertial>
-        <mass value="0.1"/>
-        <origin xyz="0 0 0" rpy="0 0 0"/>
-        <inertia ixx="0.000033" ixy="0" ixz="0" iyy="0.000033" iyz="0" izz="0.000033"/>
-    </inertial>
-</link>
-<!-- LIDAR sensor -->
-<joint name="lidar_joint" type="fixed">
-    <parent link="lidar_connector_link"/>
-    <child link="lidar_link"/>
-    <origin xyz="0 0 0.05" rpy="0 0 0"/>
-</joint>
-<link name="lidar_link">
-    <visual>
-        <origin xyz="0 0 0" rpy="0 0 0"/>
-        <geometry>
-            <cylinder radius="0.05" length="0.04"/>
-        </geometry>
-        <material name="black"/>
-    </visual>
-    <collision>
-        <origin xyz="0 0 0" rpy="0 0 0"/>
-        <geometry>
-            <cylinder radius="0.05" length="0.04"/>
-        </geometry>
-    </collision>
-    <inertial>
-        <mass value="0.1"/>
-        <origin xyz="0 0 0" rpy="0 0 0"/>
-        <inertia ixx="0.000033" ixy="0" ixz="0" iyy="0.000033" iyz="0" izz="0.000033"/>
-    </inertial>
-</link>
-<!-- ########################################################### -->
-<!-- END: LIDAR connector and sensor										 -->
-<!-- ########################################################### -->
-<!-- ########################################################### -->
-<!-- START: Camera sensor										 -->
-<!-- ########################################################### -->
-<!-- Camera sensor -->
-<joint name="camera_joint" type="fixed">
-    <parent link="body_link"/>
-    <child link="camera_link"/>
-    <origin xyz="0.5 0.05 ${body_link_z_dim/2 + 0.01}" rpy="0 0.2 0"/>  <!-- Positioned forward and slightly tilted down -->
-</joint>
-<link name="camera_link">
-    <visual>
-        <origin xyz="0 0 0" rpy="0 ${pi_const/2} 0"/>
-        <geometry>
-            <box size="0.03 0.05 0.02"/>
-        </geometry>
-        <material name="orange"/>
-    </visual>
-    <collision>
-        <origin xyz="0 0 0" rpy="0 0 0"/>
-        <geometry>
-            <box size="0.03 0.05 0.05"/>
-        </geometry>
-    </collision>
-    <inertial>
-        <mass value="0.1"/>
-        <origin xyz="0 0 0" rpy="0 0 0"/>
-        <inertia ixx="0.000033" ixy="0" ixz="0" iyy="0.000033" iyz="0" izz="0.000033"/>
-    </inertial>
-</link>
-<!-- Camera optical frame -->
-<joint name="camera_optical_joint" type="fixed">
-    <parent link="camera_link"/>
-    <child link="camera_optical_frame"/>
-    <origin xyz="0 0 0" rpy="${-pi_const/2} 0 ${-pi_const/2}"/>
-</joint>
-<link name="camera_optical_frame"/>
-<!-- ########################################################### -->
-<!-- END: Camera sensor										 -->
-<!-- ########################################################### -->
-<!-- ########################################################### -->
-<!-- START: Depth Camera sensor									 -->
-<!-- ########################################################### -->
-<!-- Depth Camera mount directly on body -->
-<joint name="depth_camera_joint" type="fixed">
-    <parent link="body_link"/>
-    <child link="depth_camera_link"/>
-    <origin xyz="0.5 -0.05 ${body_link_z_dim/2 + 0.01}" rpy="0 0.2 0"/>  <!-- Positioned forward and slightly tilted down, opposite side from camera -->
-</joint>
-<link name="depth_camera_link">
-    <visual>
-        <origin xyz="0 0 0" rpy="0 ${pi_const/2} 0"/>
-        <geometry>
-            <box size="0.03 0.05 0.02"/>
-        </geometry>
-        <material name="blue"/>
-    </visual>
-    <collision>
-        <origin xyz="0 0 0" rpy="0 0 0"/>
-        <geometry>
-            <box size="0.03 0.05 0.05"/>
-        </geometry>
-    </collision>
-    <inertial>
-        <mass value="0.1"/>
-        <origin xyz="0 0 0" rpy="0 0 0"/>
-        <inertia ixx="0.000033" ixy="0" ixz="0" iyy="0.000033" iyz="0" izz="0.000033"/>
-    </inertial>
-</link>
-<!-- Depth Camera optical frame -->
-<joint name="depth_camera_optical_joint" type="fixed">
-    <parent link="depth_camera_link"/>
-    <child link="depth_camera_optical_frame"/>
-    <origin xyz="0 0 0" rpy="${-pi_const/2} 0 ${-pi_const/2}"/>
-</joint>
-<link name="depth_camera_optical_frame"/>
-<!-- ########################################################### -->
-<!-- END: Depth Camera sensor									 -->
-<!-- ########################################################### -->
-<!-- ########################################################### -->
-<!-- START: IMU sensor                                           -->
-<!-- ########################################################### -->
-<joint name="imu_joint" type="fixed">
-    <parent link="body_link"/>
-    <child link="imu_link"/>
-    <origin xyz="0 0 ${body_link_z_dim/2 - 0.05}" rpy="0 0 0"/>
-</joint>
-<link name="imu_link">
-    <visual>
-        <origin xyz="0 0 0" rpy="0 0 0"/>
-        <geometry>
-            <box size="0.02 0.02 0.01"/>
-        </geometry>
-        <material name="red"/>
-    </visual>
-    <collision>
-        <origin xyz="0 0 0" rpy="0 0 0"/>
-        <geometry>
-            <box size="0.02 0.02 0.01"/>
-        </geometry>
-    </collision>
-    <inertial>
-        <mass value="0.01"/>
-        <origin xyz="0 0 0" rpy="0 0 0"/>
-        <inertia ixx="0.000001" ixy="0" ixz="0" iyy="0.000001" iyz="0" izz="0.000001"/>
-    </inertial>
-</link>
-<!-- ########################################################### -->
-<!-- END: IMU sensor                                             -->
-<!-- ########################################################### -->
-<!-- ########################################################### -->
-<!-- START: GPS sensor                                           -->
-<!-- ########################################################### -->
-<joint name="gps_joint" type="fixed">
-    <parent link="body_link"/>
-    <child link="gps_link"/>
-    <origin xyz="0 0 ${body_link_z_dim/2 + 0.02}" rpy="0 0 0"/>
-</joint>
-<link name="gps_link">
-    <visual>
-        <origin xyz="0 0 0" rpy="0 0 0"/>
-        <geometry>
-            <cylinder radius="0.01" length="0.01"/>
-        </geometry>
-        <material name="white"/>
-    </visual>
-    <collision>
-        <origin xyz="0 0 0" rpy="0 0 0"/>
-        <geometry>
-            <cylinder radius="0.01" length="0.01"/>
-        </geometry>
-    </collision>
-    <inertial>
-        <mass value="0.01"/>
-        <origin xyz="0 0 0" rpy="0 0 0"/>
-        <inertia ixx="0.000001" ixy="0" ixz="0" iyy="0.000001" iyz="0" izz="0.000001"/>
-    </inertial>
-</link>
-<!-- ########################################################### -->
-<!-- END: GPS sensor                                             -->
-<!-- ########################################################### -->
+<!-- INCLUDING SENSOR REFERENCES                                          -->
+<!-- ########################################################### -->
+<!-- Moved to modular file sensors/...-->
+<!-- Add modular sensors using macros -->
+<xacro:lidar_sensor parent_link="body_link" />
+<xacro:camera_sensor parent_link="body_link" x_offset="0.5" y_offset="0.05" z_offset="${body_link_z_dim/2 + 0.01}" />
+<xacro:depth_camera_sensor parent_link="body_link" x_offset="0.5" y_offset="-0.05" z_offset="${body_link_z_dim/2 + 0.01}" />
+<xacro:imu_sensor parent_link="body_link" />
+<xacro:gps_sensor parent_link="body_link" />
 </robot>

Commit message: added mapping using slam_toolbox

File: model/robot.xacro (robot description, xacro)
@@ -90,8 +90,8 @@
 <!-- ########################################################### -->
 <!-- We need to have this dummy link otherwise Gazebo will complain -->
-<link name="base_link">
+<link name="base_footprint">
 </link>
 <joint name="base_joint" type="fixed">
-	<parent link="base_link"/>
+	<parent link="base_footprint"/>
 	<child link="body_link"/>
 </joint>

Commit message: added nav2 navigation

File: model/robot.xacro (robot description, xacro)
@@ -8,14 +8,14 @@
 <robot name="differential_drive_robot" xmlns:xacro="http://www.ros.org/wiki/xacro">
 <!-- Body dimensions -->
-<xacro:property name="body_link_x_dim" value="1"/>
-<xacro:property name="body_link_y_dim" value="0.6"/>
-<xacro:property name="body_link_z_dim" value="0.3"/>
+<xacro:property name="base_link_x_dim" value="0.5"/>
+<xacro:property name="base_link_y_dim" value="0.35"/>
+<xacro:property name="base_link_z_dim" value="0.13"/>
 <!-- Wheel dimensions and locations -->
-<xacro:property name="wheel_link_radius" value="0.15"/>
-<xacro:property name="wheel_link_length" value="0.1"/>
-<xacro:property name="wheel_link_z_location" value="-0.1"/>
+<xacro:property name="wheel_link_radius" value="0.08"/>
+<xacro:property name="wheel_link_length" value="0.05"/>
+<xacro:property name="wheel_link_z_location" value="-0.05"/>
 <!-- Caster sphere dimensions and locations -->
-<xacro:property name="caster_link_radius" value="0.15"/>
-<xacro:property name="caster_link_z_location" value="-0.1"/>
+<xacro:property name="caster_link_radius" value="0.08"/>
+<xacro:property name="caster_link_z_location" value="-0.05"/>
 <!-- Material density -->
 <xacro:property name="body_density" value="2710.0"/>
@@ -25,5 +25,5 @@
 <xacro:property name="pi_const" value="3.14159265"/>
 <!-- Robot body mass, wheel mass, caster mass -->
-<xacro:property name="body_mass" value="${body_density*body_link_x_dim*body_link_y_dim*body_link_z_dim}"/>
+<xacro:property name="body_mass" value="${body_density*base_link_x_dim*base_link_y_dim*base_link_z_dim}"/>
 <xacro:property name="wheel_mass" value="${wheel_density*pi_const*wheel_link_radius*wheel_link_radius*wheel_link_length}"/>
 <xacro:property name="caster_mass" value="${caster_density*(4.0/3.0)*pi_const*caster_link_radius*caster_link_radius*caster_link_radius}"/>
@@ -75,15 +75,15 @@
     </material>
 <!-- Include the modular LIDAR sensor file -->
-<xacro:include filename="$(find mobile_dd_robot)/model/sensors/lidar.xacro" />
+<xacro:include filename="$(find danny_bot)/model/sensors/lidar.xacro" />
 <!-- Include the modular camera sensor file -->
-<xacro:include filename="$(find mobile_dd_robot)/model/sensors/camera.xacro" />
+<xacro:include filename="$(find danny_bot)/model/sensors/camera.xacro" />
 <!-- Include the modular depth camera sensor file -->
-<xacro:include filename="$(find mobile_dd_robot)/model/sensors/depth_camera.xacro" />
+<xacro:include filename="$(find danny_bot)/model/sensors/depth_camera.xacro" />
 <!-- Include the modular IMU sensor file -->
-<xacro:include filename="$(find mobile_dd_robot)/model/sensors/imu.xacro" />
+<xacro:include filename="$(find danny_bot)/model/sensors/imu.xacro" />
 <!-- Include the modular GPS sensor file -->
-<xacro:include filename="$(find mobile_dd_robot)/model/sensors/gps.xacro" />
+<xacro:include filename="$(find danny_bot)/model/sensors/gps.xacro" />
 <!-- Over here we include the file that defines extra Gazebo options and motion control driver -->
-<xacro:include filename="$(find mobile_dd_robot)/model/robot.gazebo" />
+<xacro:include filename="$(find danny_bot)/model/robot.gazebo" />
 <!-- ########################################################### -->
 <!-- FROM HERE WE DEFINE LINKS, JOINTS 				 -->
@@ -94,13 +94,13 @@
 <joint name="base_joint" type="fixed">
 	<parent link="base_footprint"/>
-	<child link="body_link"/>
+	<child link="base_link"/>
 </joint>
 <!-- ########################################################### -->
 <!-- START: Body link of the robot -->
 <!-- ########################################################### -->
-<link name="body_link">
-	<visual>
-		<geometry>
-			<box size="${body_link_x_dim} ${body_link_y_dim} ${body_link_z_dim}" />
+<link name="base_link">
+	<visual>
+		<geometry>
+			<box size="${base_link_x_dim} ${base_link_y_dim} ${base_link_z_dim}" />
 		</geometry>
 	<material name="green"/>
@@ -109,5 +109,5 @@
 	<collision>
 		<geometry>
-			<box size="${body_link_x_dim} ${body_link_y_dim} ${body_link_z_dim}" />
+			<box size="${base_link_x_dim} ${base_link_y_dim} ${base_link_z_dim}" />
 		</geometry>
 		<origin rpy="0 0 0" xyz="0 0 0"/>
@@ -117,6 +117,6 @@
 		<mass value="${body_mass}"/>
 	<inertia
-	ixx="${(1/12)*body_mass*(body_link_y_dim*body_link_y_dim+body_link_z_dim*body_link_z_dim)}" ixy="0" 		ixz="0" iyy="${(1/12)*body_mass*(body_link_x_dim*body_link_x_dim+body_link_z_dim*body_link_z_dim)}" 		iyz="0"
-	izz="${(1/12)*body_mass*(body_link_y_dim*body_link_y_dim+body_link_x_dim*body_link_x_dim)}" />
+	ixx="${(1/12)*body_mass*(base_link_y_dim*base_link_y_dim+base_link_z_dim*base_link_z_dim)}" ixy="0" 		ixz="0" iyy="${(1/12)*body_mass*(base_link_x_dim*base_link_x_dim+base_link_z_dim*base_link_z_dim)}" 		iyz="0"
+	izz="${(1/12)*body_mass*(base_link_y_dim*base_link_y_dim+base_link_x_dim*base_link_x_dim)}" />
 	</inertial>
 </link>
@@ -128,7 +128,7 @@
 <!-- ########################################################### -->
 <joint name="right_wheel_joint" type="continuous" >
-	<parent link="body_link"/>
+	<parent link="base_link"/>
 	<child  link="right_wheel_link" />
-	<origin xyz="${-2*wheel_link_radius} ${-body_link_y_dim/2-wheel_link_length/2} ${wheel_link_z_location}" rpy="0 0 0" />
+	<origin xyz="${-2*wheel_link_radius} ${-base_link_y_dim/2-wheel_link_length/2} ${wheel_link_z_location}" rpy="0 0 0" />
 	<axis xyz="0 1 0"/>
 	<limit effort="1000" velocity="1000"/>
@@ -158,7 +158,7 @@
 <!-- ########################################################### -->
 <joint name="left_wheel_joint" type="continuous" >
-	<parent link="body_link"/>
+	<parent link="base_link"/>
 	<child  link="left_wheel_link" />
-	<origin xyz="${-2*wheel_link_radius} ${body_link_y_dim/2+wheel_link_length/2} ${wheel_link_z_location}" rpy="0 0 0" />
+	<origin xyz="${-2*wheel_link_radius} ${base_link_y_dim/2+wheel_link_length/2} ${wheel_link_z_location}" rpy="0 0 0" />
 	<axis xyz="0 1 0"/>
 	<limit effort="1000" velocity="1000"/>
@@ -188,5 +188,5 @@
 <!-- ########################################################### -->
 <joint name="caster_joint" type="fixed">
-        <parent link="body_link"/>
+        <parent link="base_link"/>
         <child link="caster_link"/>
         <origin xyz="${2*caster_link_radius} 0 ${caster_link_z_location}" rpy="0 0 0"/>
@@ -216,8 +216,8 @@
 <!-- Moved to modular file sensors/...-->
 <!-- Add modular sensors using macros -->
-<xacro:lidar_sensor parent_link="body_link" />
-<xacro:camera_sensor parent_link="body_link" x_offset="0.5" y_offset="0.05" z_offset="${body_link_z_dim/2 + 0.01}" />
-<xacro:depth_camera_sensor parent_link="body_link" x_offset="0.5" y_offset="-0.05" z_offset="${body_link_z_dim/2 + 0.01}" />
-<xacro:imu_sensor parent_link="body_link" />
-<xacro:gps_sensor parent_link="body_link" />
+<xacro:lidar_sensor parent_link="base_link" />
+<xacro:camera_sensor parent_link="base_link" x_offset="0.25" y_offset="0.05" z_offset="${base_link_z_dim/2 + 0.01}" />
+<xacro:depth_camera_sensor parent_link="base_link" x_offset="0.25" y_offset="-0.05" z_offset="${base_link_z_dim/2 + 0.01}" />
+<xacro:imu_sensor parent_link="base_link" />
+<xacro:gps_sensor parent_link="base_link" />
 </robot>

File: model/sensors/gps.xacro (robot description, xacro)
@@ -6,5 +6,5 @@
         <parent link="${parent_link}"/>
         <child link="gps_link"/>
-        <origin xyz="0 0 ${body_link_z_dim/2 + 0.02}" rpy="0 0 0"/>
+        <origin xyz="0 0 ${base_link_z_dim/2 + 0.02}" rpy="0 0 0"/>
     </joint>
     <link name="gps_link">

File: model/sensors/imu.xacro (robot description, xacro)
@@ -6,5 +6,5 @@
         <parent link="${parent_link}"/>
         <child link="imu_link"/>
-        <origin xyz="0 0 ${body_link_z_dim/2 - 0.05}" rpy="0 0 0"/>
+        <origin xyz="0 0 ${base_link_z_dim/2 - 0.05}" rpy="0 0 0"/>
     </joint>
     <link name="imu_link">

File: model/sensors/lidar.xacro (robot description, xacro)
@@ -7,5 +7,5 @@
         <parent link="${parent_link}"/>
         <child link="lidar_connector_link"/>
-        <origin xyz="0 0 ${body_link_z_dim/2}" rpy="0 0 0"/>
+        <origin xyz="0 0 ${base_link_z_dim/2}" rpy="0 0 0"/>
     </joint>
     <link name="lidar_connector_link">
